File: onyx_robot.sch (KiCad schematic (older format))
At the start: 32 parts, among them P1 POWER/DOOR, P2 READER, P3 FTDI, P4 OPT, Q1 Q_NMOS_GDS, SW1 SW_PUSH, SW2 SW_PUSH, U1 ADP2301, U2 RELAY_SPDT, U3 ESP-12E

Commit message: New component for relay, pin numbering consistent with intended footprint
Parts:
- U2: symbol RELAY_SPDT -> JS_RELAY
Changed lines of the file:
@@
 LED
 $Comp
-L RELAY_SPDT U2
+L JS_RELAY U2
 U 1 1 55854FA0
 P 3775 4025

Commit message: Assign footprints
Parts:
- C1, C2: footprint (none) -> Capacitors_SMD:C_1206_HandSoldering
- C3, C4: footprint (none) -> Capacitors_SMD:C_0603_HandSoldering
- D1, D2: footprint (none) -> Diodes_SMD:Diode-SMA_Handsoldering
- L1: footprint (none) -> timhawes:LPS6225
- Q1: footprint (none) -> Housings_SOT-23_SOT-143_TSOT-6:SOT-23
- R1, R10, R11, R12, R2, R3, R4, R5, R6, R7, R8, R9: footprint (none) -> Resistors_SMD:R_0603_HandSoldering
- U1: footprint (none) -> Housings_SOT-23_SOT-143_TSOT-6:SOT-23-6
- U2: footprint (none) -> timhawes:JS_RELAY
- U3: footprint (none) -> jdunmire-kicad-ESP8266:ESP-12E
Changed lines of the file:
@@
 F 0 "U3" H 7900 4125 50  0000 C CNN
 F 1 "ESP-12E" H 7900 4325 50  0000 C CNN
-F 2 "" H 7900 4225 50  0001 C CNN
+F 2 "jdunmire-kicad-ESP8266:ESP-12E" H 7900 4225 50  0001 C CNN
 F 3 "" H 7900 4225 50  0001 C CNN
 	1    7900 4225
@@
 F 0 "R6" V 6205 4375 50  0000 C CNN
 F 1 "10K" V 6125 4375 50  0000 C CNN
-F 2 "" V 6055 4375 30  0000 C CNN
+F 2 "Resistors_SMD:R_0603_HandSoldering" V 6055 4375 30  0001 C CNN
 F 3 "" H 6125 4375 30  0000 C CNN
 	1    6125 4375
@@
 F 0 "R10" V 9205 4625 50  0000 C CNN
 F 1 "10K" V 9125 4625 50  0000 C CNN
-F 2 "" V 9055 4625 30  0000 C CNN
+F 2 "Resistors_SMD:R_0603_HandSoldering" V 9055 4625 30  0001 C CNN
 F 3 "" H 9125 4625 30  0000 C CNN
 	1    9125 4625
@@
 F 0 "P3" H 6275 2275 50  0000 C CNN
 F 1 "FTDI" V 6375 1925 50  0000 C CNN
-F 2 "" H 6275 1925 60  0000 C CNN
+F 2 "" H 6275 1925 60  0001 C CNN
 F 3 "" H 6275 1925 60  0000 C CNN
 	1    6275 1925
@@
 F 0 "P1" H 2375 7100 50  0000 C CNN
 F 1 "POWER/DOOR" V 2475 6650 50  0000 C CNN
-F 2 "" H 2375 6650 60  0000 C CNN
+F 2 "" H 2375 6650 60  0001 C CNN
 F 3 "" H 2375 6650 60  0000 C CNN
 	1    2375 6650
@@
 F 0 "P2" H 5625 7500 50  0000 C CNN
 F 1 "READER" V 5725 7050 50  0000 C CNN
-F 2 "" H 5625 7050 60  0000 C CNN
+F 2 "" H 5625 7050 60  0001 C CNN
 F 3 "" H 5625 7050 60  0000 C CNN
 	1    5625 7050
@@
 F 0 "R7" V 7405 1525 50  0000 C CNN
 F 1 "R" V 7325 1525 50  0000 C CNN
-F 2 "" V 7255 1525 30  0000 C CNN
+F 2 "Resistors_SMD:R_0603_HandSoldering" V 7255 1525 30  0001 C CNN
 F 3 "" H 7325 1525 30  0000 C CNN
 	1    7325 1525
@@
 F 0 "R8" V 7405 1925 50  0000 C CNN
 F 1 "R" V 7325 1925 50  0000 C CNN
-F 2 "" V 7255 1925 30  0000 C CNN
+F 2 "Resistors_SMD:R_0603_HandSoldering" V 7255 1925 30  0001 C CNN
 F 3 "" H 7325 1925 30  0000 C CNN
 	1    7325 1925
@@
 F 0 "SW2" H 9925 2085 50  0000 C CNN
 F 1 "SW_PUSH" H 9775 1895 50  0000 C CNN
-F 2 "" H 9775 1975 60  0000 C CNN
+F 2 "" H 9775 1975 60  0001 C CNN
 F 3 "" H 9775 1975 60  0000 C CNN
 	1    9775 1975
@@
 F 0 "R11" V 9855 1425 50  0000 C CNN
 F 1 "10K" V 9775 1425 50  0000 C CNN
-F 2 "" V 9705 1425 30  0000 C CNN
+F 2 "Resistors_SMD:R_0603_HandSoldering" V 9705 1425 30  0001 C CNN
 F 3 "" H 9775 1425 30  0000 C CNN
 	1    9775 1425
@@
 F 0 "SW1" H 8600 2085 50  0000 C CNN
 F 1 "SW_PUSH" H 8450 1895 50  0000 C CNN
-F 2 "" H 8450 1975 60  0000 C CNN
+F 2 "" H 8450 1975 60  0001 C CNN
 F 3 "" H 8450 1975 60  0000 C CNN
 	1    8450 1975
@@
 F 0 "R9" V 8530 1425 50  0000 C CNN
 F 1 "10K" V 8450 1425 50  0000 C CNN
-F 2 "" V 8380 1425 30  0000 C CNN
+F 2 "Resistors_SMD:R_0603_HandSoldering" V 8380 1425 30  0001 C CNN
 F 3 "" H 8450 1425 30  0000 C CNN
 	1    8450 1425
@@
 F 0 "R12" V 9855 4100 50  0000 C CNN
 F 1 "10K" V 9775 4100 50  0000 C CNN
-F 2 "" V 9705 4100 30  0000 C CNN
+F 2 "Resistors_SMD:R_0603_HandSoldering" V 9705 4100 30  0001 C CNN
 F 3 "" H 9775 4100 30  0000 C CNN
 	1    9775 4100
@@
 F 0 "U2" H 3775 4275 60  0000 C CNN
 F 1 "RELAY_SPDT" H 3775 3775 60  0000 C CNN
-F 2 "" H 3025 4225 60  0000 C CNN
+F 2 "timhawes:JS_RELAY" H 3025 4225 60  0001 C CNN
 F 3 "" H 3025 4225 60  0000 C CNN
 	1    3775 4025
@@
 F 0 "Q1" H 3500 4675 50  0000 R CNN
 F 1 "Q_NMOS_GDS" H 3850 4575 50  0000 R CNN
-F 2 "" H 3400 4725 29  0000 C CNN
+F 2 "Housings_SOT-23_SOT-143_TSOT-6:SOT-23" H 3400 4725 29  0001 C CNN
 F 3 "" H 3200 4625 60  0000 C CNN
 	1    3200 4625
@@
 F 0 "D2" H 3300 4125 50  0000 C CNN
 F 1 "D" H 3300 3925 50  0000 C CNN
-F 2 "" H 3300 4025 60  0000 C CNN
+F 2 "Diodes_SMD:Diode-SMA_Handsoldering" H 3300 4025 60  0001 C CNN
 F 3 "" H 3300 4025 60  0000 C CNN
 	1    3300 4025
@@
 F 0 "R5" V 3030 4825 50  0000 C CNN
 F 1 "10K" V 2950 4825 50  0000 C CNN
-F 2 "" V 2880 4825 30  0000 C CNN
+F 2 "Resistors_SMD:R_0603_HandSoldering" V 2880 4825 30  0001 C CNN
 F 3 "" H 2950 4825 30  0000 C CNN
 	1    2950 4825
@@
 F 0 "JP1" H 4550 4075 50  0000 L CNN
 F 1 "JUMPER3" H 4500 4275 50  0001 C BNN
-F 2 "" H 4500 4175 60  0000 C CNN
+F 2 "" H 4500 4175 60  0001 C CNN
 F 3 "" H 4500 4175 60  0000 C CNN
 	1    4500 4175
@@
 F 0 "U1" H 2225 1975 60  0000 C CNN
 F 1 "ADP2301" H 2225 1675 60  0000 C CNN
-F 2 "" H 2275 1475 60  0000 C CNN
+F 2 "Housings_SOT-23_SOT-143_TSOT-6:SOT-23-6" H 2275 1475 60  0001 C CNN
 F 3 "" H 2275 1475 60  0000 C CNN
 	1    2225 1525
@@
 F 0 "C1" H 1300 1525 50  0000 L CNN
 F 1 "10uF 25V" H 1075 1325 50  0000 L CNN
-F 2 "" H 1313 1275 30  0000 C CNN
+F 2 "Capacitors_SMD:C_1206_HandSoldering" H 1313 1275 30  0001 C CNN
 F 3 "" H 1275 1425 60  0000 C CNN
 	1    1275 1425
@@
 F 0 "R3" V 1655 1500 50  0000 C CNN
 F 1 "56K" V 1575 1500 50  0000 C CNN
-F 2 "" V 1505 1500 30  0000 C CNN
+F 2 "Resistors_SMD:R_0603_HandSoldering" V 1505 1500 30  0001 C CNN
 F 3 "" H 1575 1500 30  0000 C CNN
 	1    1575 1500
@@
 F 0 "R4" V 1655 2075 50  0000 C CNN
 F 1 "10K2" V 1575 2075 50  0000 C CNN
-F 2 "" V 1505 2075 30  0000 C CNN
+F 2 "Resistors_SMD:R_0603_HandSoldering" V 1505 2075 30  0001 C CNN
 F 3 "" H 1575 2075 30  0000 C CNN
 	1    1575 2075
@@
 F 0 "C3" H 2900 1475 50  0000 L CNN
 F 1 "0.1uF 6.3V" H 3000 1375 50  0000 L CNN
-F 2 "" H 2913 1225 30  0000 C CNN
+F 2 "Capacitors_SMD:C_0603_HandSoldering" H 2913 1225 30  0001 C CNN
 F 3 "" H 2875 1375 60  0000 C CNN
 	1    2875 1375
@@
 F 0 "C2" H 4050 1775 50  0000 L CNN
 F 1 "22uF 6.3V" H 4050 1575 50  0000 L CNN
-F 2 "" H 4063 1525 30  0000 C CNN
+F 2 "Capacitors_SMD:C_1206_HandSoldering" H 4063 1525 30  0001 C CNN
 F 3 "" H 4025 1675 60  0000 C CNN
 	1    4025 1675
@@
 F 0 "R1" V 3805 1675 50  0000 C CNN
 F 1 "31K6" V 3725 1675 50  0000 C CNN
-F 2 "" V 3655 1675 30  0000 C CNN
+F 2 "Resistors_SMD:R_0603_HandSoldering" V 3655 1675 30  0001 C CNN
 F 3 "" H 3725 1675 30  0000 C CNN
 	1    3725 1675
@@
 F 0 "R2" V 3805 2075 50  0000 C CNN
 F 1 "20K2" V 3725 2075 50  0000 C CNN
-F 2 "" V 3655 2075 30  0000 C CNN
+F 2 "Resistors_SMD:R_0603_HandSoldering" V 3655 2075 30  0001 C CNN
 F 3 "" H 3725 2075 30  0000 C CNN
 	1    3725 2075
@@
 F 0 "L1" V 3300 1525 50  0000 C CNN
 F 1 "4.7μH 2A" V 3450 1525 50  0000 C CNN
-F 2 "" H 3350 1525 60  0000 C CNN
+F 2 "timhawes:LPS6225" H 3350 1525 60  0001 C CNN
 F 3 "" H 3350 1525 60  0000 C CNN
 	1    3350 1525
@@
 F 0 "D1" H 2875 2175 50  0000 C CNN
 F 1 "B230A" H 2875 1975 50  0000 C CNN
-F 2 "" H 2875 2075 60  0000 C CNN
+F 2 "Diodes_SMD:Diode-SMA_Handsoldering" H 2875 2075 60  0001 C CNN
 F 3 "" H 2875 2075 60  0000 C CNN
 	1    2875 2075
@@
 F 0 "C4" H 6150 4975 50  0000 L CNN
 F 1 "0.1uF" H 6150 4775 50  0000 L CNN
-F 2 "" H 6163 4725 30  0000 C CNN
+F 2 "Capacitors_SMD:C_0603_HandSoldering" H 6163 4725 30  0001 C CNN
 F 3 "" H 6125 4875 60  0000 C CNN
 	1    6125 4875
@@
 F 0 "P4" H 4050 6950 50  0000 C CNN
 F 1 "OPT" V 4150 6700 50  0000 C CNN
-F 2 "" H 4050 6700 60  0000 C CNN
+F 2 "" H 4050 6700 60  0001 C CNN
 F 3 "" H 4050 6700 60  0000 C CNN
 	1    4050 6700
@@
 F 0 "C5" H 1325 4300 50  0000 L CNN
 F 1 "CP" H 1325 4100 50  0000 L CNN
-F 2 "" H 1338 4050 30  0000 C CNN
+F 2 "" H 1338 4050 30  0001 C CNN
 F 3 "" H 1300 4200 60  0000 C CNN
 	1    1300 4200
@@
 F 0 "C6" H 1675 4300 50  0000 L CNN
 F 1 "CP" H 1675 4100 50  0000 L CNN
-F 2 "" H 1688 4050 30  0000 C CNN
+F 2 "" H 1688 4050 30  0001 C CNN
 F 3 "" H 1650 4200 60  0000 C CNN
 	1    1650 4200

Commit message: FET and jumper added to piezo output Fix to incorrect net connection in power supply Connectors rearranged to 8+6+6 configuration Footprints assigned
Parts:
- removed C5, C6: CP, symbol CP
- removed R12: 10K, Resistors_SMD:R_0603_HandSoldering, symbol R
- removed SW1: SW_PUSH, symbol SW_PUSH
- added JP2: PROG, Pin_Headers:Pin_Header_Straight_1x02, symbol JUMPER
- added Q2: Q_NMOS_GDS, Housings_SOT-23_SOT-143_TSOT-6:SOT-23_Handsoldering, symbol Q_NMOS_GDS
- JP1: value JUMPER3 -> NO/NC; footprint (none) -> Pin_Headers:Pin_Header_Straight_1x03
- P1: value POWER/DOOR -> EXT1; footprint (none) -> timhawes:Terminal_Block_5.08mm_x6; symbol CONN_01X08 -> CONN_01X06
- P2: renamed from P4; value OPT -> EXT2; footprint (none) -> timhawes:Terminal_Block_5.08mm_x6; symbol CONN_01X04 -> CONN_01X06
- P3: renamed from P2; footprint (none) -> timhawes:Terminal_Block_5.08mm_x8
- P4: renamed from P3; footprint (none) -> Pin_Headers:Pin_Header_Straight_1x06
- Q1: footprint Housings_SOT-23_SOT-143_TSOT-6:SOT-23 -> Housings_SOT-23_SOT-143_TSOT-6:SOT-23_Handsoldering
- R1: value 31K6 -> 31K6 1%
- R2: value 20K2 -> 20K2 1%
- R3: value 56K -> 56K 1%
- R4: value 10K2 -> 10K2 1%
- R7: value R -> 10K 1%
- R8: value R -> 2K2 1%
- SW2: value SW_PUSH -> RESET; footprint (none) -> timhawes:EVQPT5
- U2: footprint timhawes:JS_RELAY -> Relays_ThroughHole:Relay_SANYOU_SRD_Series_Form_C
Connections:
- net +12V: now also P1.2 (P2); no longer P1.5 (P5)
- net +3V3: now also P3.8 (P8); no longer P3.7 (P7)
- net CLK: now also P3.2 (P2); no longer P3.1 (P1)
- net CS: now also P3.5 (P5); no longer P3.4 (P4)
- net DOOR_SENSE: now also P2.4 (P4); no longer P1.3 (P3)
- net EXIT: now also P2.2 (P2); no longer P1.1 (P1)
- net GND: now also P1.1 (P1), P1.3 (P3), P1.5 (P5), P2.1 (P1), P2.3 (P3), P2.5 (P5), P3.1 (P1), JP2.2, Q2.3 (S); no longer P1.2 (P2), P1.4 (P4), P1.6 (P6), P1.8 (P8), P2.2 (P2), P2.4 (P4), P3.8 (P8), R1.2, R2.1, U1.3 (FB)
- net LED: now also P3.6 (P6); no longer P3.5 (P5)
- net MISO: now also P3.3 (P3); no longer P3.2 (P2)
- net MOSI: now also P3.4 (P4); no longer P3.3 (P3)
- net SNIB: now also P1.6 (P6); no longer P2.1 (P1)
- net TAMPER: now also P2.6 (P6); no longer P2.3 (P3)
- net 12V_SWITCHED renamed 12V_OUT
- net 12V_OUT: now also P1.4 (P4); no longer P1.7 (P7)
- net BOOT_BUZZER renamed GPIO0
- net GPIO0: now also JP2.1, Q2.1 (G); no longer P3.6 (P6)
- new net: R1.2, R2.1, U1.3 (FB)
- new net PIEZO: P3.7 (P7), Q2.2 (D)
Other:
- note added: "GPIO0 LOW = Bootloader\nGPIO0 HIGH = Runtime"
- note added: "Measurement of 12V rail \nto detect power failures."
- moved on the sheet: C1, C2, C4, D2, JP1, P3, P4, Q1, R10, R11, R5, R6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
